File: hardware/apds9960_breakout/apds9960_breakout.kicad_pcb (KiCad board)
At the start: 2 copper layers, 26.7 x 11.4 mm, 11 parts, among them J1 Conn_01x04_Pin, J2 Conn_01x05_Pin, U1 APDS

Commit message: pin swap
Parts:
- U1: value APDS -> APDS-9960
Connections:
- J1 pad 1: SCL -> SDA
- J1 pad 2: SDA -> SCL
Routing:
- net SDA: track 26.8 -> 25.6 mm
Other:
- board text added: "EZER LONGINUS APR 2024"
- board text removed: "EZER LONGINUS MAR 2024"
