File: hardware/apds9960_breakout/apds9960_breakout.kicad_sch (KiCad schematic)
At the start: 11 parts, among them J1 Conn_01x04_Pin, J2 Conn_01x05_Pin, U1 APDS-9960

Commit message: pin swap
Connections:
- net SCL: now also J1.2 (Pin_2); no longer J1.1 (Pin_1)
- net SDA: now also J1.1 (Pin_1); no longer J1.2 (Pin_2)
Changed lines of the file:
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@@
     (effects (font (size 5.08 5.08)) (justify left bottom))
   )
-  (global_label "SDA" (shape input) (at 69.85 102.87 0) (fields_autoplaced)
+  (global_label "SDA" (shape input) (at 69.85 100.33 0) (fields_autoplaced)
     (effects (font (size 1 1)) (justify left))
-    (property "Intersheetrefs" "${INTERSHEET_REFS}" (at 75.0098 102.87 0)
+    (property "Intersheetrefs" "${INTERSHEET_REFS}" (at 75.0098 100.33 0)
       (effects (font (size 1.27 1.27)) (justify left) hide)
     )
   )
-  (global_label "SCL" (shape input) (at 69.85 100.33 0) (fields_autoplaced)
+  (global_label "SCL" (shape input) (at 69.85 102.87 0) (fields_autoplaced)
     (effects (font (size 1 1)) (justify left))
-    (property "Intersheetrefs" "${INTERSHEET_REFS}" (at 74.9622 100.33 0)
+    (property "Intersheetrefs" "${INTERSHEET_REFS}" (at 74.9622 102.87 0)
       (effects (font (size 1.27 1.27)) (justify left) hide)
     )
